File: ch32-baseboard-kicad/ch32-baseboard-kicad.kicad_sch (KiCad schematic)
At the start: 43 parts, among them J1 USB_C_USB2.0_16P, J2 TC2030, J3 53048-0310, SW1 SW_DIP_x02, SW2 TS-1088, U1 CH32V30xRxTx, U2 SPX3819M5-L-3-3, U3 INA195, X1 16MHz

Commit message: feat: silkscreen updates, manufacturing files
Parts:
- C1, C10, C11, C12, C15, C2, C4, C6, C8, C9: JLCPCB Part Number (none) -> C1525
- C13, C14: JLCPCB Part Number (none) -> C32949
- C3, C5, C7: JLCPCB Part Number (none) -> C15850
- D1, D4: JLCPCB Part Number (none) -> C7519; Manufacturer (none) -> STMicroelectronics; Manufacturer Part Number (none) -> USBLC6-2SC6
- D2: JLCPCB Part Number (none) -> C2290; Manufacturer Hubei KENTO Elec -> Hubei KENTO Elec
- D3: JLCPCB Part Number (none) -> C1976562
- J3: JLCPCB Part Number (none) -> C505275
- R1, R2: JLCPCB Part Number (none) -> C25905
- R3: JLCPCB Part Number (none) -> C17477
- R4: JLCPCB Part Number (none) -> C154638
- R5: JLCPCB Part Number (none) -> C22962
- R6, R7: JLCPCB Part Number (none) -> C25804; Manufacturer UNI-ROYAL -> UNI-ROYAL(Uniroyal Elec)
- R8: JLCPCB Part Number (none) -> C17168
- SW1: JLCPCB Part Number (none) -> C5439761
- SW2: JLCPCB Part Number (none) -> C720477
- U1: JLCPCB C2988083 -> (none); JLCPCB Part Number (none) -> C5187529; Manufacturer (none) -> WCH(Jiangsu Qin Heng); Manufacturer Part Number (none) -> CH32V305RBT6
- U2: JLCPCB Part Number (none) -> C9055
- U3: JLCPCB Part Number (none) -> C2653834; Manufacturer (none) -> Texas Instruments; Manufacturer Part Number (none) -> INA195AIDBVT
- X1: JLCPCB Part Number (none) -> C13738
